Commit message: FIXED: some syntax bug

File: gazebo_demo/robots/4limb_robot.urdf.xacro (robot description, xacro)
@@ -4,13 +4,13 @@
   <!-- The following included files set up definitions of parts of the robot body -->
   <!-- misc common stuff? -->
-  <xacro:include filename="$(find gazebo_demos)/urdf/common.xacro" />
+  <xacro:include filename="$(find gazebo_demo)/urdf/common.xacro" />
   <!-- material definition -->
-  <xacro:include filename="$(find gazebo_demos)/urdf/material.urdf.xacro" />
+  <xacro:include filename="$(find gazebo_demo)/urdf/material.urdf.xacro" />
   <!-- gazebo definition -->
-  <xacro:include filename="$(find gazebo_demos)/gazebo/gazebo.urdf.xacro" />
+  <xacro:include filename="$(find gazebo_demo)/gazebo/gazebo.urdf.xacro" />
   <!-- body definition -->
-  <xacro:include filename="$(find gazebo_demos)/urdf/body/body.urdf.xacro" />
+  <xacro:include filename="$(find gazebo_demo)/urdf/body/body.urdf.xacro" />
   <!-- limb definition -->
-  <xacro:include filename="$(find gazebo_demos)/urdf/limb/limb.urdf.xacro" />
+  <xacro:include filename="$(find gazebo_demo)/urdf/limb/limb.urdf.xacro" />
   <!-- end effector definition -->
   <!-- <xacro:include filename="$(find limbsys)/robot_description/urdf/end_effector/end_effector.urdf.xacro" /> -->
@@ -18,5 +18,6 @@
   <xacro:common/>
   <!-- body and 8 limbs -->
-  <xacro:WorldToBody name_="body"/>
+  <link name="base_link"/>
+  <xacro:BaseLinkToBody name_="body"/>
   <property name="lx" value="${0.098/2}"/>
   <property name="ly" value="${0.100/2}"/>

File: gazebo_demo/robots/8limb_robot_withEE.urdf.xacro (robot description, xacro)
@@ -1,21 +1,22 @@
 <?xml version="1.0"?>
-<robot xmlns:xacro="http://www.ros.org/wiki/xacro" name="limbsys" >
+<robot xmlns:xacro="http://www.ros.org/wiki/xacro" name="demo_robo" >
   <!-- The following included files set up definitions of parts of the robot body -->
   <!-- misc common stuff? -->
-  <xacro:include filename="$(find gazebo_demos)/urdf/common.xacro" />
+  <xacro:include filename="$(find gazebo_demo)/urdf/common.xacro" />
   <!-- material definition -->
-  <xacro:include filename="$(find gazebo_demos)/urdf/material.urdf.xacro" />
+  <xacro:include filename="$(find gazebo_demo)/urdf/material.urdf.xacro" />
   <!-- gazebo definition -->
-  <xacro:include filename="$(find gazebo_demos)/gazebo/gazebo.urdf.xacro" />
+  <xacro:include filename="$(find gazebo_demo)/gazebo/gazebo.urdf.xacro" />
   <!-- body definition -->
-  <xacro:include filename="$(find gazebo_demos)/urdf/body/body.urdf.xacro" />
+  <xacro:include filename="$(find gazebo_demo)/urdf/body/body.urdf.xacro" />
   <!-- limb definition -->
-  <xacro:include filename="$(find gazebo_demos)/urdf/limb/limb.urdf.xacro" />
+  <xacro:include filename="$(find gazebo_demo)/urdf/limb/limb.urdf.xacro" />
   <!-- end effector definition -->
-  <xacro:include filename="$(find gazebo_demos)/urdf/end_effector/end_effector.urdf.xacro" />
+  <xacro:include filename="$(find gazebo_demo)/urdf/end_effector/end_effector.urdf.xacro" />
   <!-- Now we can start using the macros included above to define our robot -->
   <xacro:common/>
   <!-- body and 8 limbs -->
-  <xacro:WorldToBody name_="body"/>
+  <link name="base_link"/>
+  <xacro:BaseLinkToBody name_="body"/>
   <property name="lx" value="0.050"/>
   <property name="ly" value="0.050"/>

File: gazebo_demo/urdf/body/body.gazebo.xacro (robot description, xacro)
@@ -1,5 +1,5 @@
 <?xml version="1.0"?>
 <robot xmlns:xacro="http://www.ros.org/wiki/xacro">
-  <xacro:macro name="WorldToBody_gazebo" params="name">
+  <xacro:macro name="BaseLinkToBody_gazebo" params="name">
     <gazebo reference="${name}">
       <material>Gazebo/Orange</material>

File: gazebo_demo/urdf/body/body.transmission.xacro (robot description, xacro)
@@ -1,5 +1,5 @@
 <?xml version="1.0"?>
 <robot xmlns:xacro="http://www.ros.org/wiki/xacro">
-  <xacro:macro name="WorldToBody_transmission" params="name">
+  <xacro:macro name="BaseLinkToBody_transmission" params="name">
 <!-- nothing -->
   </xacro:macro>

File: gazebo_demo/urdf/body/body.urdf.xacro (robot description, xacro)
@@ -1,7 +1,7 @@
 <?xml version="1.0"?>
 <robot xmlns:xacro="http://ros.org/wiki/xacro">
-  <xacro:include filename="$(find gazebo_demos)/urdf/body/body.gazebo.xacro"/>
-  <xacro:include filename="$(find gazebo_demos)/urdf/body/body.transmission.xacro"/>
-  <xacro:include filename="$(find gazebo_demos)/urdf/common.xacro"/>
+  <xacro:include filename="$(find gazebo_demo)/urdf/body/body.gazebo.xacro"/>
+  <xacro:include filename="$(find gazebo_demo)/urdf/body/body.transmission.xacro"/>
+  <xacro:include filename="$(find gazebo_demo)/urdf/common.xacro"/>
   <!-- Geometry property for box -->
   <!-- body size -->
@@ -19,11 +19,10 @@
   <property name="b_iyz" value="0"/>
   <!-- ============= Body Description ============= -->
-  <!-- baselinkToBody is better? -->
-  <xacro:macro name="WorldToBody" params="name_">
-      <joint name="jointwb" type="floating">
-        <parent link="world"/>
-        <child link="${name_}"/>
-        <origin xyz="0 0 0" rpy="0 0 0"/>
-      </joint>
+  <xacro:macro name="BaseLinkToBody" params="name_">
+    <joint name="jointblTobody" type="fixed">
+      <parent link="base_link"/>
+      <child link="${name_}"/>
+      <origin xyz="0 0 0" rpy="0 0 0"/>
+    </joint>
     <!-- central body -->
     <link name="${name_}">
@@ -49,6 +48,6 @@
       </collision>
     </link>
-    <xacro:WorldToBody_gazebo name="${name_}" />
-    <xacro:WorldToBody_transmission name="${name_}" />
+    <xacro:BaseLinkToBody_gazebo name="${name_}" />
+    <xacro:BaseLinkToBody_transmission name="${name_}" />
   </xacro:macro>
 </robot>

File: gazebo_demo/urdf/common.xacro (robot description, xacro)
@@ -1,18 +1,15 @@
 <?xml version="1.0"?>
 <robot xmlns:xacro="http://ros.org/wiki/xacro">
-	<property name="M_PI" value="3.1415926535897931" />
-	<property name="VELOCITY_LIMIT_SCALE" value="0.6" />
-	<!-- motor information -->
-	<property name="dx_lo" value="-${150*M_PI/180}" />
-	<property name="dx_up" value="+${150*M_PI/180}" />
-	<property name="dx_eff" value="3.621866" />
-	<property name="dx_vel" value="7.016224" />
-	<!-- Mathmatic -->
-	<property name="Sin45" value="0.707106781"/>
-	<property name="Cos45" value="0.707106781"/>
-	<xacro:macro name="common">
-<!--
-		<link name="world"/>
--->
-	</xacro:macro>
+  <property name="M_PI" value="3.1415926535897931" />
+  <property name="VELOCITY_LIMIT_SCALE" value="0.6" />
+  <!-- motor information -->
+  <property name="dx_lo" value="-${150*M_PI/180}" />
+  <property name="dx_up" value="+${150*M_PI/180}" />
+  <property name="dx_eff" value="3.621866" />
+  <property name="dx_vel" value="7.016224" />
+  <!-- Mathmatic -->
+  <property name="Sin45" value="0.707106781"/>
+  <property name="Cos45" value="0.707106781"/>
+  <xacro:macro name="common">
+  </xacro:macro>
 </robot>

File: gazebo_demo/urdf/limb/limb.urdf.xacro (robot description, xacro)
@@ -3,5 +3,5 @@
 <robot xmlns:xacro="http://www.ros.org/wiki/xacro">
   <xacro:include filename="$(find gazebo_demo)/urdf/limb/limb.gazebo.xacro"/>
-  <xacro:include filename="$(find gazebo_demo)/urdf/limb/limb.transmission_position.xacro"/>
+  <xacro:include filename="$(find gazebo_demo)/urdf/limb/limb.transmission.xacro"/>
   <xacro:include filename="$(find gazebo_demo)/urdf/common.xacro"/>
   <!-- length and radius property of cylinder link of a limb -->
