Commit message: ADDED: gazebo launch

File: gazebo_demo/urdf/material.urdf.xacro (robot description, xacro)
@@ -1,24 +1,21 @@
 <?xml version="1.0"?>
 <robot xmlns:xacro="http://ros.org/wiki/xacro">
-	<material name="Cyan">
-		<color rgba="0.0 0.0 1.0 1.0"/>
-	</material>
-	<material name="Blue">
-		<color rgba="0.0 0.0 0.8 1.0"/>
-	</material>
-	<material name="Green">
-		<color rgba="0.0 0.8 0.0 1.0"/>
-	</material>
-	<material name="Red">
-		<color rgba="0.8 0.0 0.0 1.0"/>
-	</material>
-	<material name="White">
-		<color rgba="1.0 1.0 1.0 1.0"/>
-	</material>
-	<material name="Yellow">
-		<color rgba="1.0 1.0 0.0 1.0"/>
-	</material>
-<!-- 	<material name="image">
-		<texture filename="package://limbsys/robot_description/textures/~.png"/>
-	</material> -->
+  <material name="Cyan">
+    <color rgba="0.0 0.0 1.0 1.0"/>
+  </material>
+  <material name="Blue">
+    <color rgba="0.0 0.0 0.8 1.0"/>
+  </material>
+  <material name="Green">
+    <color rgba="0.0 0.8 0.0 1.0"/>
+  </material>
+  <material name="Red">
+    <color rgba="0.8 0.0 0.0 1.0"/>
+  </material>
+  <material name="White">
+    <color rgba="1.0 1.0 1.0 1.0"/>
+  </material>
+  <material name="Yellow">
+    <color rgba="1.0 1.0 0.0 1.0"/>
+  </material>
 </robot>
