Commit message: FIXED: some deprecated syntax

File: gazebo_demo/urdf/body/body.gazebo.xacro (robot description, xacro)
@@ -1,4 +1,4 @@
 <?xml version="1.0"?>
-<robot xmlns:xacro="http://www.ros.org/wiki/xacro">
+<robot xmlns:xacro="http://ros.org/wiki/xacro">
   <xacro:macro name="BaseLinkToBody_gazebo" params="name">
     <gazebo reference="${name}">

File: gazebo_demo/urdf/body/body.transmission.xacro (robot description, xacro)
@@ -1,4 +1,4 @@
 <?xml version="1.0"?>
-<robot xmlns:xacro="http://www.ros.org/wiki/xacro">
+<robot xmlns:xacro="http://ros.org/wiki/xacro">
   <xacro:macro name="BaseLinkToBody_transmission" params="name">
 <!-- nothing -->

File: gazebo_demo/urdf/body/body.urdf.xacro (robot description, xacro)
@@ -6,16 +6,16 @@
   <!-- Geometry property for box -->
   <!-- body size -->
-  <property name="b_x" value="0.100"/>
-  <property name="b_y" value="0.100"/>
-  <property name="b_z" value="0.100"/>
+  <xacro:property name="b_x" value="0.100"/>
+  <xacro:property name="b_y" value="0.100"/>
+  <xacro:property name="b_z" value="0.100"/>
   <!-- body mass -->
-  <property name="b_m" value="0.300"/>
+  <xacro:property name="b_m" value="0.300"/>
   <!-- inertia tensol -->
-  <property name="b_ixx" value="${(1/12)*b_m*(b_y*b_y+b_z*b_z)}"/>
-  <property name="b_iyy" value="${(1/12)*b_m*(b_x*b_x+b_z*b_z)}"/>
-  <property name="b_izz" value="${(1/12)*b_m*(b_x*b_x+b_y*b_y)}"/>
-  <property name="b_ixy" value="0"/>
-  <property name="b_ixz" value="0"/>
-  <property name="b_iyz" value="0"/>
+  <xacro:property name="b_ixx" value="${(1/12)*b_m*(b_y*b_y+b_z*b_z)}"/>
+  <xacro:property name="b_iyy" value="${(1/12)*b_m*(b_x*b_x+b_z*b_z)}"/>
+  <xacro:property name="b_izz" value="${(1/12)*b_m*(b_x*b_x+b_y*b_y)}"/>
+  <xacro:property name="b_ixy" value="0"/>
+  <xacro:property name="b_ixz" value="0"/>
+  <xacro:property name="b_iyz" value="0"/>
   <!-- ============= Body Description ============= -->
   <xacro:macro name="BaseLinkToBody" params="name_">

File: gazebo_demo/urdf/common.xacro (robot description, xacro)
@@ -1,14 +1,14 @@
 <?xml version="1.0"?>
 <robot xmlns:xacro="http://ros.org/wiki/xacro">
-  <property name="M_PI" value="3.1415926535897931" />
-  <property name="VELOCITY_LIMIT_SCALE" value="0.6" />
+  <xacro:property name="M_PI" value="3.1415926535897931" />
+  <xacro:property name="VELOCITY_LIMIT_SCALE" value="0.6" />
   <!-- motor information -->
-  <property name="dx_lo" value="-${150*M_PI/180}" />
-  <property name="dx_up" value="+${150*M_PI/180}" />
-  <property name="dx_eff" value="3.621866" />
-  <property name="dx_vel" value="7.016224" />
+  <xacro:property name="dx_lo" value="-${150*M_PI/180}" />
+  <xacro:property name="dx_up" value="+${150*M_PI/180}" />
+  <xacro:property name="dx_eff" value="3.621866" />
+  <xacro:property name="dx_vel" value="7.016224" />
   <!-- Mathmatic -->
-  <property name="Sin45" value="0.707106781"/>
-  <property name="Cos45" value="0.707106781"/>
+  <xacro:property name="Sin45" value="0.707106781"/>
+  <xacro:property name="Cos45" value="0.707106781"/>
   <xacro:macro name="common">
   </xacro:macro>

File: gazebo_demo/urdf/end_effector/end_effector.gazebo.xacro (robot description, xacro)
@@ -1,4 +1,4 @@
 <?xml version="1.0"?>
-<robot xmlns:xacro="http://www.ros.org/wiki/xacro">
+<robot xmlns:xacro="http://ros.org/wiki/xacro">
   <xacro:macro name="EE_gazebo" params="limbNo_g">
     <gazebo reference="EEbase_${limbNo_g}">

File: gazebo_demo/urdf/end_effector/end_effector.transmission.xacro (robot description, xacro)
@@ -1,4 +1,4 @@
 <?xml version="1.0"?>
-<robot xmlns:xacro="http://www.ros.org/wiki/xacro">
+<robot xmlns:xacro="http://ros.org/wiki/xacro">
   <xacro:macro name="EE_transmission" params="limbNo_t">
     <!-- EE_up -->

File: gazebo_demo/urdf/end_effector/end_effector.urdf.xacro (robot description, xacro)
@@ -1,5 +1,5 @@
 <?xml version="1.0"?>
 <!-- XML namespaces -->
-<robot xmlns:xacro="http://www.ros.org/wiki/xacro">
+<robot xmlns:xacro="http://ros.org/wiki/xacro">
   <xacro:include filename="$(find gazebo_demo)/urdf/end_effector/end_effector.gazebo.xacro"/>
   <xacro:include filename="$(find gazebo_demo)/urdf/end_effector/end_effector.transmission.xacro"/>
@@ -7,51 +7,51 @@
   <!-- length and radius property of cylinder link of a limb -->
   <!-- EE_base -->
-  <property name="Eb_x"   value="0.010" />
-  <property name="Eb_y"   value="0.030" />
-  <property name="Eb_z"   value="${0.030+0.002}" /> <!-- 1mm margin -->
-  <property name="Eb_m"   value="0.050"/>
-  <property name="Eb_ixx" value="${(1/12)*Eb_m*(Eb_y*Eb_y+Eb_z*Eb_z)}"/>
-  <property name="Eb_iyy" value="${(1/12)*Eb_m*(Eb_x*Eb_x+Eb_z*Eb_z)}"/>
-  <property name="Eb_izz" value="${(1/12)*Eb_m*(Eb_x*Eb_x+Eb_y*Eb_y)}"/>
-  <property name="Eb_ixy" value="0" />
-  <property name="Eb_ixz" value="0" />
-  <property name="Eb_iyz" value="0" />
+  <xacro:property name="Eb_x"   value="0.010" />
+  <xacro:property name="Eb_y"   value="0.030" />
+  <xacro:property name="Eb_z"   value="${0.030+0.002}" /> <!-- 1mm margin -->
+  <xacro:property name="Eb_m"   value="0.050"/>
+  <xacro:property name="Eb_ixx" value="${(1/12)*Eb_m*(Eb_y*Eb_y+Eb_z*Eb_z)}"/>
+  <xacro:property name="Eb_iyy" value="${(1/12)*Eb_m*(Eb_x*Eb_x+Eb_z*Eb_z)}"/>
+  <xacro:property name="Eb_izz" value="${(1/12)*Eb_m*(Eb_x*Eb_x+Eb_y*Eb_y)}"/>
+  <xacro:property name="Eb_ixy" value="0" />
+  <xacro:property name="Eb_ixz" value="0" />
+  <xacro:property name="Eb_iyz" value="0" />
   <!-- EE_up -->
-  <property name="Eu_x"   value="0.050" />
-  <property name="Eu_y"   value="0.030" />
-  <property name="Eu_z"   value="0.010" />
-  <property name="Eu_m"   value="0.050"/>
-  <property name="Eu_ixx" value="${(1/12)*Eu_m*(Eu_y*Eu_y+Eu_z*Eu_z)}"/>
-  <property name="Eu_iyy" value="${(1/12)*Eu_m*(Eu_x*Eu_x+Eu_z*Eu_z)}"/>
-  <property name="Eu_izz" value="${(1/12)*Eu_m*(Eu_x*Eu_x+Eu_y*Eu_y)}"/>
-  <property name="Eu_ixy" value="0" />
-  <property name="Eu_ixz" value="0" />
-  <property name="Eu_iyz" value="0" />
-  <property name="Eu_up"  value="+${10*M_PI/180}"/>
-  <property name="Eu_lo"  value="-${M_PI/2 + 5 *M_PI/180}"/>
+  <xacro:property name="Eu_x"   value="0.050" />
+  <xacro:property name="Eu_y"   value="0.030" />
+  <xacro:property name="Eu_z"   value="0.010" />
+  <xacro:property name="Eu_m"   value="0.050"/>
+  <xacro:property name="Eu_ixx" value="${(1/12)*Eu_m*(Eu_y*Eu_y+Eu_z*Eu_z)}"/>
+  <xacro:property name="Eu_iyy" value="${(1/12)*Eu_m*(Eu_x*Eu_x+Eu_z*Eu_z)}"/>
+  <xacro:property name="Eu_izz" value="${(1/12)*Eu_m*(Eu_x*Eu_x+Eu_y*Eu_y)}"/>
+  <xacro:property name="Eu_ixy" value="0" />
+  <xacro:property name="Eu_ixz" value="0" />
+  <xacro:property name="Eu_iyz" value="0" />
+  <xacro:property name="Eu_up"  value="+${10*M_PI/180}"/>
+  <xacro:property name="Eu_lo"  value="-${M_PI/2 + 5 *M_PI/180}"/>
   <!-- EE_down -->
-  <property name="Ed_x"   value="0.025" />
-  <property name="Ed_y"   value="0.030" />
-  <property name="Ed_z"   value="0.010" />
-  <property name="Ed_m"   value="0.050"/>
-  <property name="Ed_ixx" value="${(1/12)*Ed_m*(Ed_y*Ed_y+Ed_z*Ed_z)}"/>
-  <property name="Ed_iyy" value="${(1/12)*Ed_m*(Ed_x*Ed_x+Ed_z*Ed_z)}"/>
-  <property name="Ed_izz" value="${(1/12)*Ed_m*(Ed_x*Ed_x+Ed_y*Ed_y)}"/>
-  <property name="Ed_ixy" value="0" />
-  <property name="Ed_ixz" value="0" />
-  <property name="Ed_iyz" value="0" />
-  <property name="Ed_up"  value="+${M_PI/2}"/>
-  <property name="Ed_lo"  value="-${10*M_PI/180}"/>
+  <xacro:property name="Ed_x"   value="0.025" />
+  <xacro:property name="Ed_y"   value="0.030" />
+  <xacro:property name="Ed_z"   value="0.010" />
+  <xacro:property name="Ed_m"   value="0.050"/>
+  <xacro:property name="Ed_ixx" value="${(1/12)*Ed_m*(Ed_y*Ed_y+Ed_z*Ed_z)}"/>
+  <xacro:property name="Ed_iyy" value="${(1/12)*Ed_m*(Ed_x*Ed_x+Ed_z*Ed_z)}"/>
+  <xacro:property name="Ed_izz" value="${(1/12)*Ed_m*(Ed_x*Ed_x+Ed_y*Ed_y)}"/>
+  <xacro:property name="Ed_ixy" value="0" />
+  <xacro:property name="Ed_ixz" value="0" />
+  <xacro:property name="Ed_iyz" value="0" />
+  <xacro:property name="Ed_up"  value="+${M_PI/2}"/>
+  <xacro:property name="Ed_lo"  value="-${10*M_PI/180}"/>
   <!-- EE_nail -->
-  <property name="En_x"   value="0.010" />
-  <property name="En_y"   value="0.030" />
-  <property name="En_z"   value="0.010" />
-  <property name="En_m"   value="0.020" />
-  <property name="En_ixx" value="${(1/12)*En_m*(En_y*En_y+En_z*En_z)}"/>
-  <property name="En_iyy" value="${(1/12)*En_m*(En_x*En_x+En_z*En_z)}"/>
-  <property name="En_izz" value="${(1/12)*En_m*(En_x*En_x+En_y*En_y)}"/>
-  <property name="En_ixy" value="0" />
-  <property name="En_ixz" value="0" />
-  <property name="En_iyz" value="0" />
+  <xacro:property name="En_x"   value="0.010" />
+  <xacro:property name="En_y"   value="0.030" />
+  <xacro:property name="En_z"   value="0.010" />
+  <xacro:property name="En_m"   value="0.020" />
+  <xacro:property name="En_ixx" value="${(1/12)*En_m*(En_y*En_y+En_z*En_z)}"/>
+  <xacro:property name="En_iyy" value="${(1/12)*En_m*(En_x*En_x+En_z*En_z)}"/>
+  <xacro:property name="En_izz" value="${(1/12)*En_m*(En_x*En_x+En_y*En_y)}"/>
+  <xacro:property name="En_ixy" value="0" />
+  <xacro:property name="En_ixz" value="0" />
+  <xacro:property name="En_iyz" value="0" />
   <!-- ============ EE Description ============ -->
   <xacro:macro name="EE_gripper" params="limbNo parent px py pz prow ppit pyaw">

File: gazebo_demo/urdf/limb/limb.gazebo.xacro (robot description, xacro)
@@ -1,4 +1,4 @@
 <?xml version="1.0"?>
-<robot xmlns:xacro="http://www.ros.org/wiki/xacro">
+<robot xmlns:xacro="http://ros.org/wiki/xacro">
   <xacro:macro name="limb4_gazebo" params="limbNo_g">
     <gazebo reference="link${limbNo_g}_1">
@@ -14,5 +14,5 @@
     <gazebo reference="link${limbNo_g}_3">
       <selfCollide>true</selfCollide>
-        <mu1>0.5</mu1>
+      <mu1>0.5</mu1>
       <mu2>0.5</mu2>
     </gazebo>

File: gazebo_demo/urdf/limb/limb.transmission.xacro (robot description, xacro)
@@ -1,4 +1,4 @@
 <?xml version="1.0"?>
-<robot xmlns:xacro="http://www.ros.org/wiki/xacro">
+<robot xmlns:xacro="http://ros.org/wiki/xacro">
   <xacro:macro name="limb4_transmission" params="limbNo_t">
     <transmission name="tran${limbNo_t}_01">

File: gazebo_demo/urdf/limb/limb.urdf.xacro (robot description, xacro)
@@ -1,5 +1,5 @@
 <?xml version="1.0"?>
 <!-- XML namespaces -->
-<robot xmlns:xacro="http://www.ros.org/wiki/xacro">
+<robot xmlns:xacro="http://ros.org/wiki/xacro">
   <xacro:include filename="$(find gazebo_demo)/urdf/limb/limb.gazebo.xacro"/>
   <xacro:include filename="$(find gazebo_demo)/urdf/limb/limb.transmission.xacro"/>
@@ -7,43 +7,43 @@
   <!-- length and radius property of cylinder link of a limb -->
   <!-- link1 -->
-  <property name="l1_length" value="0.094" />
-  <property name="l1_radius" value="0.015" />
-  <property name="l1_mass"   value="0.2"/>
-  <property name="l1_ixx"    value="${(1/4)*l1_mass*l1_radius*l1_radius+(1/12)*l1_mass*l1_length*l1_length}"/>
-  <property name="l1_iyy"    value="${(1/4)*l1_mass*l1_radius*l1_radius+(1/12)*l1_mass*l1_length*l1_length}"/>
-  <property name="l1_izz"    value="${(1/2)*l1_mass*l1_radius*l1_radius}"/>
-  <property name="l1_ixy"    value="0" />
-  <property name="l1_ixz"    value="0" />
-  <property name="l1_iyz"    value="0" />
+  <xacro:property name="l1_length" value="0.094" />
+  <xacro:property name="l1_radius" value="0.015" />
+  <xacro:property name="l1_mass"   value="0.2"/>
+  <xacro:property name="l1_ixx"    value="${(1/4)*l1_mass*l1_radius*l1_radius+(1/12)*l1_mass*l1_length*l1_length}"/>
+  <xacro:property name="l1_iyy"    value="${(1/4)*l1_mass*l1_radius*l1_radius+(1/12)*l1_mass*l1_length*l1_length}"/>
+  <xacro:property name="l1_izz"    value="${(1/2)*l1_mass*l1_radius*l1_radius}"/>
+  <xacro:property name="l1_ixy"    value="0" />
+  <xacro:property name="l1_ixz"    value="0" />
+  <xacro:property name="l1_iyz"    value="0" />
   <!-- link2 -->
-  <property name="l2_length" value="0.095" />
-  <property name="l2_radius" value="0.015" />
-  <property name="l2_mass"   value="0.2"/>
-  <property name="l2_ixx"    value="${(1/4)*l2_mass*l2_radius*l2_radius+(1/12)*l2_mass*l2_length*l2_length}"/>
-  <property name="l2_iyy"    value="${(1/4)*l2_mass*l2_radius*l2_radius+(1/12)*l2_mass*l2_length*l2_length}"/>
-  <property name="l2_izz"    value="${(1/2)*l2_mass*l2_radius*l2_radius}"/>
-  <property name="l2_ixy"    value="0" />
-  <property name="l2_ixz"    value="0" />
-  <property name="l2_iyz"    value="0" />
+  <xacro:property name="l2_length" value="0.095" />
+  <xacro:property name="l2_radius" value="0.015" />
+  <xacro:property name="l2_mass"   value="0.2"/>
+  <xacro:property name="l2_ixx"    value="${(1/4)*l2_mass*l2_radius*l2_radius+(1/12)*l2_mass*l2_length*l2_length}"/>
+  <xacro:property name="l2_iyy"    value="${(1/4)*l2_mass*l2_radius*l2_radius+(1/12)*l2_mass*l2_length*l2_length}"/>
+  <xacro:property name="l2_izz"    value="${(1/2)*l2_mass*l2_radius*l2_radius}"/>
+  <xacro:property name="l2_ixy"    value="0" />
+  <xacro:property name="l2_ixz"    value="0" />
+  <xacro:property name="l2_iyz"    value="0" />
   <!-- link3 -->
-  <property name="l3_length" value="0.099" />
-  <property name="l3_radius" value="0.015" />
-  <property name="l3_mass"   value="0.2"/>
-  <property name="l3_ixx"    value="${(1/4)*l3_mass*l3_radius*l3_radius+(1/12)*l3_mass*l3_length*l3_length}"/>
-  <property name="l3_iyy"    value="${(1/4)*l3_mass*l3_radius*l3_radius+(1/12)*l3_mass*l3_length*l3_length}"/>
-  <property name="l3_izz"    value="${(1/2)*l3_mass*l3_radius*l3_radius}"/>
-  <property name="l3_ixy"    value="0" />
-  <property name="l3_ixz"    value="0" />
-  <property name="l3_iyz"    value="0" />
+  <xacro:property name="l3_length" value="0.099" />
+  <xacro:property name="l3_radius" value="0.015" />
+  <xacro:property name="l3_mass"   value="0.2"/>
+  <xacro:property name="l3_ixx"    value="${(1/4)*l3_mass*l3_radius*l3_radius+(1/12)*l3_mass*l3_length*l3_length}"/>
+  <xacro:property name="l3_iyy"    value="${(1/4)*l3_mass*l3_radius*l3_radius+(1/12)*l3_mass*l3_length*l3_length}"/>
+  <xacro:property name="l3_izz"    value="${(1/2)*l3_mass*l3_radius*l3_radius}"/>
+  <xacro:property name="l3_ixy"    value="0" />
+  <xacro:property name="l3_ixz"    value="0" />
+  <xacro:property name="l3_iyz"    value="0" />
   <!-- link4 -->
-  <property name="l4_length" value="0.140" />
-  <property name="l4_radius" value="0.015" />
-  <property name="l4_mass"   value="0.2"/>
-  <property name="l4_ixx"    value="${(1/4)*l4_mass*l4_radius*l4_radius+(1/12)*l4_mass*l4_length*l4_length}"/>
-  <property name="l4_iyy"    value="${(1/4)*l4_mass*l4_radius*l4_radius+(1/12)*l4_mass*l4_length*l4_length}"/>
-  <property name="l4_izz"    value="${(1/2)*l4_mass*l4_radius*l4_radius}"/>
-  <property name="l4_ixy"    value="0" />
-  <property name="l4_ixz"    value="0" />
-  <property name="l4_iyz"    value="0" />
+  <xacro:property name="l4_length" value="0.140" />
+  <xacro:property name="l4_radius" value="0.015" />
+  <xacro:property name="l4_mass"   value="0.2"/>
+  <xacro:property name="l4_ixx"    value="${(1/4)*l4_mass*l4_radius*l4_radius+(1/12)*l4_mass*l4_length*l4_length}"/>
+  <xacro:property name="l4_iyy"    value="${(1/4)*l4_mass*l4_radius*l4_radius+(1/12)*l4_mass*l4_length*l4_length}"/>
+  <xacro:property name="l4_izz"    value="${(1/2)*l4_mass*l4_radius*l4_radius}"/>
+  <xacro:property name="l4_ixy"    value="0" />
+  <xacro:property name="l4_ixz"    value="0" />
+  <xacro:property name="l4_iyz"    value="0" />
   <!-- ============= Limb Description ============= -->
   <xacro:macro name="link_limb4" params="limbNo parent px py pz prow ppit pyaw">
