Commit message: FIXED: some deprecated, too

File: gazebo_demo/urdf/end_effector/end_effector.transmission.xacro (robot description, xacro)
@@ -6,8 +6,8 @@
       <type>transmission_interface/SimpleTransmission</type>
       <joint name="joint${limbNo_t}_bu">
-        <hardwareInterface>EffortJointInterface</hardwareInterface>
+        <hardwareInterface>hardware_interface/EffortJointInterface</hardwareInterface>
       </joint>
       <actuator name="motor${limbNo_t}_bu">
-        <hardwareInterface>EffortJointInterface</hardwareInterface>
+        <hardwareInterface>hardware_interface/EffortJointInterface</hardwareInterface>
         <mechanicalReduction>1</mechanicalReduction>
       </actuator>
@@ -17,8 +17,8 @@
       <type>transmission_interface/SimpleTransmission</type>
       <joint name="joint${limbNo_t}_bd">
-        <hardwareInterface>EffortJointInterface</hardwareInterface>
+        <hardwareInterface>hardware_interface/EffortJointInterface</hardwareInterface>
       </joint>
       <actuator name="motor${limbNo_t}_bd">
-        <hardwareInterface>EffortJointInterface</hardwareInterface>
+        <hardwareInterface>hardware_interface/EffortJointInterface</hardwareInterface>
         <mechanicalReduction>1</mechanicalReduction>
       </actuator>

File: gazebo_demo/urdf/limb/limb.gazebo.xacro (robot description, xacro)
@@ -22,44 +22,4 @@
       <mu2>0.5</mu2>
     </gazebo>
-    <gazebo reference="joint${limbNo_g}_01">
-      <erp>0.1</erp>
-      <stopKd value="1000000000.0" />
-      <stopKp value="1000000000.0" />
-      <fudgeFactor value="0.5" />
-      <cfmDamping>true</cfmDamping>
-      <axis>
-        <dynamics damping="0.7" friction="0"/>
-      </axis>
-    </gazebo>
-    <gazebo reference="joint${limbNo_g}_12">
-      <erp>0.1</erp>
-      <stopKd value="1000000000.0" />
-      <stopKp value="1000000000.0" />
-      <fudgeFactor value="0.5" />
-      <cfmDamping>true</cfmDamping>
-      <axis>
-        <dynamics damping="0.7" friction="0"/>
-      </axis>
-    </gazebo>
-    <gazebo reference="joint${limbNo_g}_23">
-      <erp>0.1</erp>
-      <stopKd value="1000000000.0" />
-      <stopKp value="1000000000.0" />
-      <fudgeFactor value="0.5" />
-      <cfmDamping>true</cfmDamping>
-      <axis>
-        <dynamics damping="0.7" friction="0"/>
-      </axis>
-    </gazebo>
-    <gazebo reference="joint${limbNo_g}_34">
-      <erp>0.1</erp>
-      <stopKd value="1000000000.0" />
-      <stopKp value="1000000000.0" />
-      <fudgeFactor value="0.5" />
-      <cfmDamping>true</cfmDamping>
-      <axis>
-        <dynamics damping="0.7" friction="0"/>
-      </axis>
-    </gazebo>
   </xacro:macro>
 </robot>

File: gazebo_demo/urdf/limb/limb.transmission.xacro (robot description, xacro)
@@ -5,8 +5,8 @@
       <type>transmission_interface/SimpleTransmission</type>
       <joint name="joint${limbNo_t}_01">
-        <hardwareInterface>EffortJointInterface</hardwareInterface>
+        <hardwareInterface>hardware_interface/EffortJointInterface</hardwareInterface>
       </joint>
       <actuator name="motor${limbNo_t}_01">
-        <hardwareInterface>EffortJointInterface</hardwareInterface>
+        <hardwareInterface>hardware_interface/EffortJointInterface</hardwareInterface>
         <mechanicalReduction>1</mechanicalReduction>
       </actuator>
@@ -15,8 +15,8 @@
       <type>transmission_interface/SimpleTransmission</type>
       <joint name="joint${limbNo_t}_12">
-        <hardwareInterface>EffortJointInterface</hardwareInterface>
+        <hardwareInterface>hardware_interface/EffortJointInterface</hardwareInterface>
       </joint>
       <actuator name="motor${limbNo_t}_12">
-        <hardwareInterface>EffortJointInterface</hardwareInterface>
+        <hardwareInterface>hardware_interface/EffortJointInterface</hardwareInterface>
         <mechanicalReduction>1</mechanicalReduction>
       </actuator>
@@ -25,8 +25,8 @@
       <type>transmission_interface/SimpleTransmission</type>
       <joint name="joint${limbNo_t}_23">
-        <hardwareInterface>EffortJointInterface</hardwareInterface>
+        <hardwareInterface>hardware_interface/EffortJointInterface</hardwareInterface>
       </joint>
       <actuator name="motor${limbNo_t}_23">
-        <hardwareInterface>EffortJointInterface</hardwareInterface>
+        <hardwareInterface>hardware_interface/EffortJointInterface</hardwareInterface>
         <mechanicalReduction>1</mechanicalReduction>
       </actuator>
@@ -35,8 +35,8 @@
       <type>transmission_interface/SimpleTransmission</type>
       <joint name="joint${limbNo_t}_34">
-        <hardwareInterface>EffortJointInterface</hardwareInterface>
+        <hardwareInterface>hardware_interface/EffortJointInterface</hardwareInterface>
       </joint>
       <actuator name="motor${limbNo_t}_34">
-        <hardwareInterface>EffortJointInterface</hardwareInterface>
+        <hardwareInterface>hardware_interface/EffortJointInterface</hardwareInterface>
         <mechanicalReduction>1</mechanicalReduction>
       </actuator>
